Commit message: Working lower arm

File: urdf/luko.urdf (robot description, URDF)
Before this commit: robot luko, 6 links, 5 joints
Links:
- link link3: geometry visual box size=0.01 0.05 0.05
Joints:
- joint joint0: origin xyz=0 0 0 rpy=0 0 0 -> xyz=0 -0.02 0.125 rpy=0 0 0
- joint joint1: origin xyz=0 0.5 0 rpy=0 0 0 -> xyz=0 0.02 0.125 rpy=0 0 0
- joint joint2: origin xyz=0 0 0.5 rpy=0 0 0 -> xyz=0 0 0.25 rpy=0 0 0

Commit message: Working both arms and rotating base, head not modelled yet

File: urdf/luko.urdf (robot description, URDF)
Before this commit: robot luko, 6 links, 5 joints
Links:
- removed link link1
- removed link link2
- removed link link3
- removed link lower_link
- added link bottom_mount; visual box size=0.01 0.05 0.05
- added link head_mount; visual box size=0.01 0.05 0.05
- added link low_aft_rod; visual cylinder length=0.25 radius=0.005
- added link low_fwd_rod; visual cylinder length=0.25 radius=0.005
- added link middle_piece; visual box size=0.01 0.05 0.05
- added link up_aft_rod; visual cylinder length=0.25 radius=0.005
- added link up_fwd_rod; visual cylinder length=0.25 radius=0.005
Joints:
- removed joint joint0
- removed joint joint1
- removed joint joint2
- added joint low_joint0: type revolute, parent bottom_mount, child low_fwd_rod, origin xyz=0 -0.02 0.125 rpy=0 0 0, axis 1 0 0, limit lower=-1.57 upper=1.57 effort=0.5293 velocity=6.159937255
- added joint low_joint1: type revolute, parent bottom_mount, child low_aft_rod, origin xyz=0 0.02 0.125 rpy=0 0 0, axis 1 0 0, limit lower=-1.57 upper=1.57 effort=0.5293 velocity=6.159937255, mimic joint=low_joint0 multiplier=1 offset=0
- added joint low_joint2: type revolute, parent low_fwd_rod, child middle_piece, origin xyz=0 0 0.25 rpy=0 0 0, axis 1 0 0, limit lower=-1.57 upper=1.57 effort=0.5293 velocity=6.159937255, mimic joint=low_joint0 multiplier=-1 offset=0
- added joint up_joint0: type revolute, parent middle_piece, child up_fwd_rod, origin xyz=0 0 0 rpy=0 0 0, axis 1 0 0, limit lower=-1.57 upper=1.57 effort=0.5293 velocity=6.159937255
- added joint up_joint1: type revolute, parent middle_piece, child up_aft_rod, origin xyz=0 0 0.045 rpy=0 0 0, axis 1 0 0, limit lower=-1.57 upper=1.57 effort=0.5293 velocity=6.159937255, mimic joint=up_joint0 multiplier=1 offset=0
- added joint up_joint2: type revolute, parent up_fwd_rod, child head_mount, origin xyz=0 -0.25 0 rpy=0 0 0, axis 1 0 0, limit lower=-1.57 upper=1.57 effort=0.5293 velocity=6.159937255, mimic joint=up_joint0 multiplier=-1 offset=0
- joint cylinder_joint: axis (none) -> 0 0 1; child lower_link -> bottom_mount; limit (none) -> lower=-3.14 upper=3.14 effort=0.5293 velocity=6.159937255; type fixed -> revolute

Commit message: initial mostly accurate model

File: urdf/luko.urdf (robot description, URDF)
Before this commit: robot luko, 9 links, 8 joints
Links:
- added link head_aft; visual cylinder length=0.07 radius=0.025
- added link head_fwd; visual cylinder length=0.05 radius=0.05
- added link head_link; visual cylinder length=0.02 radius=0.004
- link head_mount: geometry visual box size=0.01 0.03 0.03
- link low_aft_rod: geometry visual cylinder length=0.22 radius=0.005
- link low_fwd_rod: geometry visual cylinder length=0.22 radius=0.005
- link up_aft_rod: geometry visual cylinder length=0.17 radius=0.005
- link up_fwd_rod: geometry visual cylinder length=0.17 radius=0.005
Joints:
- added joint head_bearing_link: type revolute, parent head_mount, child head_link, origin xyz=0 -0.02 0.005 rpy=0 0 0, axis 1 0 0, limit lower=-1.57 upper=1.57 effort=0.5293 velocity=6.159937255
- added joint head_to_lamp: type fixed, parent head_link, child head_aft, origin xyz=0 0 0 rpy=0 0 0
- added joint head_to_reflector: type fixed, parent head_aft, child head_fwd, origin xyz=0 0 0 rpy=0 0 0
- joint low_joint0: origin xyz=0 -0.02 0.125 rpy=0 0 0 -> xyz=0 -0.0145 0.085 rpy=-0.38 0 0
- joint low_joint1: origin xyz=0 0.02 0.125 rpy=0 0 0 -> xyz=0 0.0145 0.100 rpy=-0.30 0 0
- joint low_joint2: origin xyz=0 0 0.25 rpy=0 0 0 -> xyz=0 0 0.22 rpy=0 0 0
- joint up_joint0: origin xyz=0 0 0 rpy=0 0 0 -> xyz=0 -0.01 0 rpy=0.38 0 0
- joint up_joint1: origin xyz=0 0 0.045 rpy=0 0 0 -> xyz=0 -0.025 0.01 rpy=0.38 0 0
- joint up_joint2: origin xyz=0 -0.25 0 rpy=0 0 0 -> xyz=0 -0.165 -0.005 rpy=0 0 0

Commit message: Motion planning package and basic poses

File: urdf/luko.urdf (robot description, URDF)
Before this commit: robot luko, 12 links, 11 joints
Joints:
- joint head_to_lamp: axis (none) -> 0 -1 0; limit (none) -> lower=-1.57 upper=1.57 effort=0.5293 velocity=6.159937255; type fixed -> revolute
